File: pcb/led-controller.kicad_pcb (KiCad board)
At the start: 4 copper layers, 0 parts

Commit message: Progress on STM32F411 wiring
Parts:
- added C1: 10uF, Capacitor_SMD:C_0603_1608Metric, F.Cu at (149.0, 122.8)
- added C10: 10nF, Capacitor_SMD:C_0603_1608Metric, F.Cu at (166.5, 105.0)
- added C11: 1uF, Capacitor_SMD:C_0603_1608Metric, F.Cu at (137.0, 123.1)
- added C12: 1uF, Capacitor_SMD:C_0603_1608Metric, F.Cu at (145.0, 123.1)
- added C13: 1uF, Capacitor_SMD:C_0603_1608Metric, F.Cu at (111.3, 113.0)
- added C2: 10pF, Capacitor_SMD:C_0603_1608Metric, F.Cu at (146.1, 115.2)
- added C3: 100nF, Capacitor_SMD:C_0603_1608Metric, F.Cu at (158.9, 112.0)
- added C4: 10pF, Capacitor_SMD:C_0603_1608Metric, F.Cu at (141.0, 125.6)
- added C5: 100nF, Capacitor_SMD:C_0603_1608Metric, F.Cu at (141.0, 123.1)
- added C6: 100nF, Capacitor_SMD:C_0603_1608Metric, F.Cu at (145.0, 125.6)
- added C7: 4u7F, Capacitor_SMD:C_0603_1608Metric, F.Cu at (162.5, 105.0)
- added C8: 100nF, Capacitor_SMD:C_0603_1608Metric, F.Cu at (137.0, 120.6)
- added C9: 100nF, Capacitor_SMD:C_0603_1608Metric, F.Cu at (162.9, 110.0)
- added H1: MountingHole_Pad, MountingHole:MountingHole_2.2mm_M2_Pad, F.Cu at (131.5, 111.5)
- added H3: MountingHole_Pad, MountingHole:MountingHole_2.2mm_M2_Pad, F.Cu at (119.5, 111.5)
- added J1: BOOT_SEL, Connector_PinHeader_1.27mm:PinHeader_1x03_P1.27mm_Horizontal, F.Cu at (151.5, 105.8)
- added J2: Programmer Conn, Connector:Tag-Connect_TC2030-IDC-FP_2x03_P1.27mm_Vertical, F.Cu at (145.7, 93.2)
- added J3: USB_C_Receptacle, Connector_USB:USB_C_Receptacle_Amphenol_12401548E4-2A, F.Cu at (96.5, 111.8)
- added R1: 4.7k, Resistor_SMD:R_0603_1608Metric, F.Cu at (154.9, 110.9)
- added R10: 100k, Resistor_SMD:R_0603_1608Metric, B.Cu at (108.0, 116.0)
- added R11: 4.7k, Resistor_SMD:R_0603_1608Metric, F.Cu at (137.0, 125.6)
- added R12: 10k, Resistor_SMD:R_0603_1608Metric, B.Cu at (103.4, 116.0)
- added R13: 100k, Resistor_SMD:R_0603_1608Metric, B.Cu at (109.5, 116.0)
- added R2: 10k, Resistor_SMD:R_0603_1608Metric, F.Cu at (158.9, 109.5)
- added R3: 22R, Resistor_SMD:R_0603_1608Metric, F.Cu at (104.3, 109.0)
- added R4: 22R, Resistor_SMD:R_0603_1608Metric, F.Cu at (104.3, 107.5)
- added R5: 10k, Resistor_SMD:R_0603_1608Metric, F.Cu at (143.1, 100.3)
- added R6: 470R, Resistor_SMD:R_0603_1608Metric, F.Cu at (111.3, 110.0)
- added R7: 1k, Resistor_SMD:R_0603_1608Metric, F.Cu at (111.3, 111.5)
- added R8: 4.7k, Resistor_SMD:R_0603_1608Metric, F.Cu at (162.9, 107.5)
- added R9: 10k, Resistor_SMD:R_0603_1608Metric, B.Cu at (105.0, 116.0)
- added SW1: PD Reset, Button_Switch_SMD:SW_SPST_B3U-1000P, F.Cu at (150.0, 111.8)
- added U1: STM32F411CCUx, Package_DFN_QFN:QFN-48-1EP_7x7mm_P0.5mm_EP5.6x5.6mm, F.Cu at (142.4, 108.4)
- added U2: STUSB4500QTR, Package_DFN_QFN:QFN-24-1EP_4x4mm_P0.5mm_EP2.7x2.7mm, F.Cu at (107.0, 113.0)
- added Y1: 16MHz, Crystal:Crystal_SMD_Abracon_ABM8G-4Pin_3.2x2.5mm, F.Cu at (157.9, 106.0)

Commit message: PCB updates
Parts:
- removed J1: BOOT_SEL, Connector_PinHeader_1.27mm:PinHeader_1x03_P1.27mm_Horizontal
- removed R3, R4: 22R, Resistor_SMD:R_0603_1608Metric
- added C14: 1uF, Capacitor_SMD:C_0603_1608Metric, F.Cu at (133.8, 102.8)
- added C15: 1uF, Capacitor_SMD:C_0603_1608Metric, F.Cu at (133.8, 100.2)
- added C16: 1uF, Capacitor_SMD:C_0603_1608Metric, F.Cu at (121.7, 102.5)
- added C17: 100nF, Capacitor_SMD:C_0603_1608Metric, F.Cu at (126.9, 97.7)
- added F1: 5A, ATL:Littlefuse-154, F.Cu at (108.2, 105.8)
- added Q1: AONR21321, ATL:AONR21321, F.Cu at (121.9, 99.0)
- added R14: 1k, Resistor_SMD:R_0603_1608Metric, F.Cu at (129.7, 100.2)
- added R15: 100k, Resistor_SMD:R_0603_1608Metric, F.Cu at (125.7, 102.5)
- added R16: 22k, Resistor_SMD:R_0603_1608Metric, F.Cu at (130.9, 97.7)
- added R17: 100R, Resistor_SMD:R_0603_1608Metric, F.Cu at (129.7, 102.8)
- added SW2: BOOT SEL, Button_Switch_SMD:SW_DIP_SPSTx01_Slide_Copal_CVS-01xB_W5.9mm_P1mm, B.Cu at (154.4, 100.6)
- R1: moved to B.Cu
- moved R1 47.5 mm to (107.4, 109.8)
- moved J3 1.56 mm to (96.4, 110.2)
Connections:
- U1 pad 32: Net-(R3-Pad1) -> D-
- U1 pad 33: Net-(R4-Pad1) -> D+
- U2 pad 16: unconnected-(U2-Pad16) -> Net-(U2-Pad16)
- U2 pad 21: unconnected-(U2-Pad21) -> Net-(U2-Pad21)
- U2 pad 23: unconnected-(U2-Pad23) -> +2V7
- U2 pad 24: GND -> VBUS
- U2 pad 9: unconnected-(U2-Pad9) -> Net-(U2-Pad9)
