File: pcb/led-controller.kicad_sch (KiCad schematic)
At the start: 0 parts

Commit message: WIP STUSB4500 (USB-C PD IC)
Parts:
- added C?: 1uF, symbol Device:C_Small
- added D?: Dual Zenner ESD Protection, symbol Device:D_Zener_Dual_CommonAnode_KKA_Parallel
- added D?: D_Schottky, symbol Device:D_Schottky
- added F?: 5A, symbol Device:Fuse
- added J?: USB_C_Receptacle, symbol Connector:USB_C_Receptacle
- added R? (x2): 10k, symbol Device:R_Small_US
- added R?: 470R, symbol Device:R_Small_US
- added R? (x2): 100k, symbol Device:R_Small_US
- added R?: 1k, symbol Device:R_Small_US
- added SW?: PD Reset, symbol Switch:SW_Push
- added U?: STM32F411CCUx, Package_DFN_QFN:QFN-48-1EP_7x7mm_P0.5mm_EP5.6x5.6mm, symbol MCU_ST_STM32F4:STM32F411CCUx
- added U?: STUSB4500QTR, Package_DFN_QFN:QFN-24-1EP_4x4mm_P0.5mm_EP2.7x2.7mm, symbol Interface_USB:STUSB4500QTR
Connections:
- new net: R?.1, R?.2, SW?.1
- new net: R?.2, U?.6 (RESET)
- new net: D?.1 (K), J?.A5 (CC1), U?.1 (CC1DB), U?.2 (CC1)
- new net: D?.2 (K), J?.B5 (CC2), U?.4 (CC2), U?.5 (CC2DB)
- new net: F?.1, J?.A4 (VBUS), J?.A9 (VBUS), J?.B4 (VBUS), J?.B9 (VBUS)
- new net: C?.1, D?.1 (K), R?.1, R?.2
- new net: R?.2, U?.12 (ADDR0)
- new net: R?.2, U?.13 (ADDR1)
- new net: R?.2, U?.18 (VBUS_VS_DISCH)
- new net +3V3: SW?.2
- new net D+: J?.A6 (D+), J?.B6 (D+)
- new net D-: J?.A7 (D-), J?.B7 (D-)
- new net Earth: J?.S1 (SHIELD)
- new net GND: C?.2, D?.3 (A), J?.A1 (GND), J?.A12 (GND), J?.B1 (GND), J?.B12 (GND), R?.1, R?.1, R?.1, U?.10 (GND), U?.22 (VSYS), U?.24 (VDD), U?.25 (GND)
- new net SCL_0: U?.7 (SCL)
- new net SDA_0: U?.8 (SDA)
- new net VBUS: D?.2 (A), F?.2, R?.1
- no-connect marks 0 -> 10

Commit message: Progress on STM32F411 wiring
Parts:
- added C1: 10uF, Capacitor_SMD:C_0603_1608Metric, symbol Device:C_Small
- added C10: 10nF, Capacitor_SMD:C_0603_1608Metric, symbol Device:C_Small
- added C11, C12: 1uF, Capacitor_SMD:C_0603_1608Metric, symbol Device:C_Small
- added C2, C4: 10pF, Capacitor_SMD:C_0603_1608Metric, symbol Device:C_Small
- added C3, C5, C6, C8, C9: 100nF, Capacitor_SMD:C_0603_1608Metric, symbol Device:C_Small
- added C7: 4u7F, Capacitor_SMD:C_0603_1608Metric, symbol Device:C_Small
- added FB1: 120R, symbol Device:FerriteBead_Small
- added H1, H3: MountingHole_Pad, MountingHole:MountingHole_2.2mm_M2_Pad, symbol Mechanical:MountingHole_Pad
- added J1: BOOT_SEL, Connector_PinHeader_1.27mm:PinHeader_1x03_P1.27mm_Horizontal, symbol Connector_Generic:Conn_01x03
- added J2: Programmer Conn, Connector:Tag-Connect_TC2030-IDC-FP_2x03_P1.27mm_Vertical, symbol ATL:TC2030
- added R1, R11, R8: 4.7k, Resistor_SMD:R_0603_1608Metric, symbol Device:R_Small_US
- added R2, R5: 10k, Resistor_SMD:R_0603_1608Metric, symbol Device:R_Small_US
- added R3, R4: 22R, Resistor_SMD:R_0603_1608Metric, symbol Device:R_Small_US
- added Y1: 16MHz, Crystal:Crystal_SMD_Abracon_ABM8G-4Pin_3.2x2.5mm, symbol Device:Crystal_GND24_Small
- C13: renamed from C?; footprint (none) -> Capacitor_SMD:C_0603_1608Metric
- J3: renamed from J?; footprint (none) -> Connector_USB:USB_C_Receptacle_Amphenol_12401548E4-2A
- R10, R12, R13, R6, R7, R9: renamed from R?; footprint (none) -> Resistor_SMD:R_0603_1608Metric
- SW1: renamed from SW?; footprint (none) -> Button_Switch_SMD:SW_SPST_B3U-1000P
- gave numbers to parts that had none: 5
Connections:
- net +3V3 is gone; now on net +3.3V: SW1.2
- net SCL_0 is gone; now on net I2C1_SCL: U2.7 (SCL)
- net SDA_0 is gone; now on net I2C1_SDA: U2.8 (SDA)
- net D+: now also R4.2
- net D-: now also R3.2
- net GND: now also U1.23 (VSS), U1.35 (VSS), U1.47 (VSS), U1.49 (VSS), U1.8 (VSSA), C1.2, C10.2, C11.2, C12.2, C2.2, C3.2, C4.2, C5.2, C6.1, C7.1, C8.2, C9.2, J1.3 (Pin_3), J2.5 (GND), Y1.2, Y1.4
- net +3.3V: now reaches U1.1 (VBAT)
- net +3.3V: now also U1.24 (VDD), U1.36 (VDD), U1.48 (VDD), C1.1, C12.1, C3.1, C5.1, C8.1, C9.1, FB1.2, J1.1 (Pin_1), R1.1, R11.1, R8.1
- net UART2_TX: now reaches U1.12 (PA2)
- net UART2_RX: now reaches U1.13 (PA3)
- net SPI_CLK: now reaches U1.15 (PA5)
- net SDIO_CMD: now reaches U1.16 (PA6)
- net SPI_MOSI: now reaches U1.17 (PA7)
- net PD_ALERT: now reaches U1.21 (PB10)
- net PD_ALERT: now also U2.19 (ALERT), R1.2
- net at U1.22 (VCAP1): now also C7.2
- net UART1_RX: now reaches U1.31 (PA10)
- net at U1.32 (PA11): now also R3.1
- net at U1.33 (PA12): now also R4.1
- net SWDIO: now reaches U1.34 (PA13)
- net SWDIO: now also J2.2 (SWDIO)
- net SWO: now reaches U1.39 (PB3)
- net SWO: now also J2.6 (SWO)
- net SPI_MISO: now reaches U1.40 (PB4)
- net SDIO_D3: now reaches U1.41 (PB5)
- net UART1_TX: now reaches U1.42 (PB6)
- net SDIO_D0: now reaches U1.43 (PB7)
- net at U1.44 (BOOT0): now also R2.2
- net I2C1_SCL: now reaches U1.45 (PB8)
- net I2C1_SCL: now also R8.2
- net I2C1_SDA: now reaches U1.46 (PB9)
- net I2C1_SDA: now also R11.2
- net at U1.5 (PH0): now also C2.1, Y1.1
- net at U1.6 (PH1): now also C4.1, Y1.3
- net ~{RESET}: now reaches U1.7 (NRST)
- net ~{RESET}: now also C6.2, R5.1
- net +3.3VA: now reaches U1.9 (VDDA)
- net +3.3VA: now also C10.1, C11.1, FB1.1
- new net: J1.2 (Pin_2), R2.1
- new net: J2.3 (~{RESET}), R5.2
- new net SWCLK: J2.4 (SWCLK)
- no-connect marks 10 -> 16
Other:
- moved on the sheet: C13, D1, D2, F1, J3, R10, R12, R13, R6, R7, R9, SW1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

Commit message: PCB updates
Parts:
- removed J1: BOOT_SEL, Connector_PinHeader_1.27mm:PinHeader_1x03_P1.27mm_Horizontal, symbol Connector_Generic:Conn_01x03
- removed R3, R4: 22R, Resistor_SMD:R_0603_1608Metric, symbol Device:R_Small_US
- added C14, C15, C16: 1uF, Capacitor_SMD:C_0603_1608Metric, symbol Device:C_Small
- added C17: 100nF, Capacitor_SMD:C_0603_1608Metric, symbol Device:C_Small
- added D3: TVS Uni 22V, symbol Device:D_Zener
- added Q1: AONR21321, ATL:AONR21321, symbol ATL:AONR21321
- added R14: 1k, Resistor_SMD:R_0603_1608Metric, symbol Device:R_Small_US
- added R15: 100k, Resistor_SMD:R_0603_1608Metric, symbol Device:R_Small_US
- added R16: 22k, Resistor_SMD:R_0603_1608Metric, symbol Device:R_Small_US
- added R17: 100R, Resistor_SMD:R_0603_1608Metric, symbol Device:R_Small_US
- added SW2: BOOT SEL, Button_Switch_SMD:SW_DIP_SPSTx01_Slide_Copal_CVS-01xB_W5.9mm_P1mm, symbol Switch:SW_Push_SPDT
- D1: value Dual Zenner ESD Protection -> Dual Uni TVS ESD
- F1: footprint (none) -> ATL:Littlefuse-154
Connections:
- net +3.3V: now also SW2.1 (A)
- net D+: now also U1.33 (PA12)
- net D-: now also U1.32 (PA11)
- net GND: now also C14.2, C15.2, C16.2, D3.2 (A), SW2.3 (C); no longer U2.24 (VDD)
- net VBUS: now also U2.24 (VDD), C14.1, Q1.1 (S), R15.1
- net at R2.1: now also SW2.2 (B)
- net at U2.16 (VBUS_EN_SNK): now also R16.2
- net at U2.21 (VREG_1V2): now also C16.1
- net +2V7: now reaches U2.23 (VREG_2V7)
- net +2V7: now also C15.1
- net at U2.9 (DISCH): now also R14.1
- new net: Q1.2 (G), R15.2, R16.1, R17.1
- new net: C17.2, R17.2
- new net VDD: C17.1, D3.1 (K), Q1.3 (D), R14.2
- no-connect marks 16 -> 20
Other:
- note added: "MCU - STM32F411"
- note added: "USB-C PD Power Regulation"
- moved on the sheet: C1, C10, C11, C12, C13, C2, C3, C4, C5, C6, C7, C8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
